Commit message: add mjcf

File: urdf/__bl_biped.urdf (robot description, URDF)
Before this commit: robot __bl_biped, 11 links, 10 joints
Links:
- link base_link: geometry collision mesh filename=package://practice_biped_robot/meshes/base_link.STL; visual mesh filename=package://practice_biped_robot/meshes/base_link.STL
- link foot_left: geometry collision mesh filename=package://practice_biped_robot/meshes/foot_left.STL; visual mesh filename=package://practice_biped_robot/meshes/foot_left.STL
- link foot_right: geometry collision mesh filename=package://practice_biped_robot/meshes/foot_right.STL; visual mesh filename=package://practice_biped_robot/meshes/foot_right.STL
- link hip_aa_left_side_bl_biped: geometry collision mesh filename=package://practice_biped_robot/meshes/hip_aa_left_side_bl_b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; visual mesh filename=package://practice_biped_robot/meshes/hip_aa_left_side_bl_b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
- link hip_aa_right_side_bl_biped: geometry collision mesh filename=package://practice_biped_robot/meshes/hip_aa_right_side_bl_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; visual mesh filename=package://practice_biped_robot/meshes/hip_aa_right_side_bl_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
- link hip_fe_left_side_bl_biped: geometry collision mesh filename=package://practice_biped_robot/meshes/hip_fe_left_side_bl_b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; visual mesh filename=package://practice_biped_robot/meshes/hip_fe_left_side_bl_b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
- link hip_fe_right_side_bl_biped: geometry collision mesh filename=package://practice_biped_robot/meshes/hip_fe_right_side_bl_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; visual mesh filename=package://practice_biped_robot/meshes/hip_fe_right_side_bl_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
- link lower_leg_left: geometry collision mesh filename=package://practice_biped_robot/meshes/lower_leg_left.STL; visual mesh filename=package://practice_biped_robot/meshes/lower_leg_left.STL
- link lower_leg_right: geometry collision mesh filename=package://practice_biped_robot/meshes/lower_leg_right.STL; visual mesh filename=package://practice_biped_robot/meshes/lower_leg_right.STL
- link upper_leg_left: geometry collision mesh filename=package://practice_biped_robot/meshes/upper_leg_left.STL; visual mesh filename=package://practice_biped_robot/meshes/upper_leg_left.STL
- link upper_leg_right: geometry collision mesh filename=package://practice_biped_robot/meshes/upper_leg_right.STL; visual mesh filename=package://practice_biped_robot/meshes/upper_leg_right.STL
